File: nexapad.kicad_sch (KiCad schematic)
At the start: 0 parts

Commit message: Finished the PCB
Parts:
- added D1, D2, D3, D4, D5, D6, D7, D8, D9: 1N4148, Diode_THT:D_DO-35_SOD27_P7.62mm_Horizontal, symbol Diode:1N4148
- added SSD1306_OLED1: ~, CustomStuff:SSD1306-0.91-OLED, symbol CustomStuff:SSD1306-0.91-OLED
- added SW1, SW2, SW4, SW5, SW6, SW7, SW8, SW9: SW_Push_45deg, Button_Switch_Keyboard:SW_Cherry_MX_1.00u_PCB, symbol Switch:SW_Push_45deg
- added SW3: RotaryEncoder_Switch, RotaryEncoder:RotaryEncoder_Alps_EC11E-Switch_Vertical_H20mm, symbol Device:RotaryEncoder_Switch
- added U1: XIAO-RP2040-DIP, OPL:XIAO-RP2040-DIP, symbol OPL:XIAO-RP2040-DIP
Connections:
- new net: D9.2 (A), SW9.2
- new net: D8.2 (A), SW8.2
- new net: D6.2 (A), SW6.2
- new net: D4.2 (A), SW4.2
- new net: SSD1306_OLED1.3 (SCL), U1.6 (GPIO7/SCL)
- new net: SSD1306_OLED1.4 (SDA), U1.5 (GPIO6/SDA)
- new net: D5.2 (A), SW5.2
- new net: D1.2 (A), SW1.2
- new net: D2.2 (A), SW2.2
- new net: D7.2 (A), SW7.2
- new net: D3.2 (A), SW3.S1
- new net +3V3: SSD1306_OLED1.2 (VCC), U1.12 (3V3)
- new net COL1: SW1.1, SW4.1, SW7.1, U1.11 (GPIO3/MOSI)
- new net COL2: SW2.1, SW5.1, SW8.1, U1.10 (GPIO4/MISO)
- new net COL3: SW3.S2, SW6.1, SW9.1, U1.9 (GPIO2/SCK)
- new net GND: SSD1306_OLED1.1 (GND), SW3.C, U1.13 (GND)
- new net ROW1: D1.1 (K), D2.1 (K), D3.1 (K), U1.1 (GPIO26/ADC0/A0)
- new net ROW2: D4.1 (K), D5.1 (K), D6.1 (K), U1.2 (GPIO27/ADC1/A1)
- new net ROW3: D7.1 (K), D8.1 (K), D9.1 (K), U1.3 (GPIO28/ADC2/A2)
- new net R_ENC_A: SW3.A, U1.7 (GPIO0/TX)
- new net R_ENC_B: SW3.B, U1.8 (GPIO1/RX)
